Commit message: bicycle model ros2_control works w gazebo

File: description/robot.urdf.xacro (robot description, xacro)
@@ -1,7 +1,12 @@
 <?xml version="1.0"?>
 <robot xmlns:xacro="http://www.ros.org/wiki/xacro"  name="robot">
-    <!-- Example link -->
-    <xacro:include filename="robot_core.xacro"/>
-        <!-- Example link -->
-    <link name="base_link"></link>
+<xacro:arg name="prefix" default="" />
+ <xacro:include filename="carlikebot_description.urdf.xacro" />
+  <!-- Import Rviz colors -->
+  <xacro:include filename="carlikebot.materials.xacro" />
+  <!-- Import carlikebot ros2_control description -->
+  <xacro:include filename="carlikebot.ros2_control.xacro" />
+  <xacro:carlikebot prefix="$(arg prefix)" />
+  <xacro:carlikebot_ros2_control
+    name="CarlikeBot" prefix="$(arg prefix)" />
 </robot>
